File: PCB/fidget.sch (KiCad schematic (older format))
At the start: 88 parts, among them J1 KEYSTONE 120, J2 KEYSTONE 120, U1 MCP73831-2ACI/MC, U10 SLG46140, U2 ESP8285, U3 TLV70033DSE, U4 LIS2DE, U5 TPS60150, U6 TPS60150, U7 TPS60150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

Commit message: moved hall sensor to battery rail so it can work with the LDO powered off
Connections:
- net +3V3: no longer C23.1, R14.2, R15.1
- net +BATT: now also C23.1, R14.2, R15.1
- net ENL: now also U10.14 (GPIO); no longer U10.13 (GPIO)
- net IDX: no longer R15.2, U8.2 (Q)
- new net IDX1: R15.2, U10.13 (GPIO), U8.2 (Q)
- no-connect marks 19 -> 18
Changed lines of the file:
@@
 Connection ~ 1200 1300
 Text Label 8850 2550 2    60   ~ 0
-IDX
+IDX1
 Wire Wire Line
 	8550 2450 8550 2550
@@
 $EndComp
 $Comp
-L +3V3 #PWR062
-U 1 1 593BA402
-P 8550 2150
-F 0 "#PWR062" H 8550 2000 50  0001 C CNN
-F 1 "+3V3" H 8550 2290 50  0000 C CNN
-F 2 "" H 8550 2150 50  0001 C CNN
-F 3 "" H 8550 2150 50  0001 C CNN
-	1    8550 2150
-	1    0    0    -1
-$EndComp
-$Comp
-L +3V3 #PWR063
-U 1 1 593BA4C8
-P 7700 2150
-F 0 "#PWR063" H 7700 2000 50  0001 C CNN
-F 1 "+3V3" H 7700 2290 50  0000 C CNN
-F 2 "" H 7700 2150 50  0001 C CNN
-F 3 "" H 7700 2150 50  0001 C CNN
-	1    7700 2150
-	1    0    0    -1
-$EndComp
-$Comp
 L C C23
 U 1 1 593C099C
@@
 $EndComp
 $Comp
-L +3V3 #PWR064
-U 1 1 593C09A2
-P 8150 1900
-F 0 "#PWR064" H 8150 1750 50  0001 C CNN
-F 1 "+3V3" H 8150 2040 50  0000 C CNN
-F 2 "" H 8150 1900 50  0001 C CNN
-F 3 "" H 8150 1900 50  0001 C CNN
-	1    8150 1900
-	1    0    0    -1
-$EndComp
-$Comp
-L GND #PWR065
+L GND #PWR062
 U 1 1 593C09A8
 P 8150 2200
-F 0 "#PWR065" H 8150 1950 50  0001 C CNN
+F 0 "#PWR062" H 8150 1950 50  0001 C CNN
 F 1 "GND" H 8150 2050 50  0000 C CNN
 F 2 "" H 8150 2200 50  0001 C CNN
@@
 $EndComp
 $Comp
-L GND #PWR066
+L GND #PWR063
 U 1 1 593C31CF
 P 7050 2300
-F 0 "#PWR066" H 7050 2050 50  0001 C CNN
+F 0 "#PWR063" H 7050 2050 50  0001 C CNN
 F 1 "GND" H 7050 2150 50  0000 C CNN
 F 2 "" H 7050 2300 50  0001 C CNN
@@
 $EndComp
 $Comp
-L +5C #PWR067
+L +5C #PWR064
 U 1 1 593D1A67
 P 1800 3300
-F 0 "#PWR067" H 1800 3150 50  0001 C CNN
+F 0 "#PWR064" H 1800 3150 50  0001 C CNN
 F 1 "+5C" H 1800 3440 50  0000 C CNN
 F 2 "" H 1800 3300 50  0001 C CNN
@@
 $EndComp
 $Comp
-L +3V3 #PWR068
+L +3V3 #PWR065
 U 1 1 593D1DEC
 P 800 3300
-F 0 "#PWR068" H 800 3150 50  0001 C CNN
+F 0 "#PWR065" H 800 3150 50  0001 C CNN
 F 1 "+3V3" H 800 3440 50  0000 C CNN
 F 2 "" H 800 3300 50  0001 C CNN
@@
 $EndComp
 $Comp
-L GND #PWR069
+L GND #PWR066
 U 1 1 593D1EA7
 P 1800 3700
-F 0 "#PWR069" H 1800 3450 50  0001 C CNN
+F 0 "#PWR066" H 1800 3450 50  0001 C CNN
 F 1 "GND" H 1800 3550 50  0000 C CNN
 F 2 "" H 1800 3700 50  0001 C CNN
@@
 $EndComp
 $Comp
-L GND #PWR070
+L GND #PWR067
 U 1 1 593FDF0A
 P 10900 3400
-F 0 "#PWR070" H 10900 3150 50  0001 C CNN
+F 0 "#PWR067" H 10900 3150 50  0001 C CNN
 F 1 "GND" H 10900 3250 50  0000 C CNN
 F 2 "" H 10900 3400 50  0001 C CNN
@@
 $EndComp
 $Comp
-L +BATT #PWR071
+L +BATT #PWR068
 U 1 1 593FE01B
 P 10900 3100
-F 0 "#PWR071" H 10900 2950 50  0001 C CNN
+F 0 "#PWR068" H 10900 2950 50  0001 C CNN
 F 1 "+BATT" H 10900 3240 50  0000 C CNN
 F 2 "" H 10900 3100 50  0001 C CNN
@@
 $EndComp
 $Comp
-L +BATT #PWR072
+L +BATT #PWR069
 U 1 1 593FE2F0
 P 9400 3000
-F 0 "#PWR072" H 9400 2850 50  0001 C CNN
+F 0 "#PWR069" H 9400 2850 50  0001 C CNN
 F 1 "+BATT" H 9400 3140 50  0000 C CNN
 F 2 "" H 9400 3000 50  0001 C CNN
@@
 $EndComp
 $Comp
-L GND #PWR073
+L GND #PWR070
 U 1 1 593FE403
 P 10300 3600
-F 0 "#PWR073" H 10300 3350 50  0001 C CNN
+F 0 "#PWR070" H 10300 3350 50  0001 C CNN
 F 1 "GND" H 10300 3450 50  0000 C CNN
 F 2 "" H 10300 3600 50  0001 C CNN
@@
 Wire Wire Line
 	10550 3300 10300 3300
-Text Label 10550 3100 2    60   ~ 0
+Text Label 10550 3000 2    60   ~ 0
 ENL
 Wire Wire Line
@@
 NoConn ~ 9400 3600
 Wire Wire Line
-	10550 3100 10300 3100
-NoConn ~ 10300 3000
+	10550 3000 10300 3000
 NoConn ~ 9400 3300
 NoConn ~ 4900 1800
 NoConn ~ 9400 3100
+$Comp
+L +BATT #PWR071
+U 1 1 593FCFD7
+P 7700 2150
+F 0 "#PWR071" H 7700 2000 50  0001 C CNN
+F 1 "+BATT" H 7700 2290 50  0000 C CNN
+F 2 "" H 7700 2150 50  0001 C CNN
+F 3 "" H 7700 2150 50  0001 C CNN
+	1    7700 2150
+	1    0    0    -1
+$EndComp
+$Comp
+L +BATT #PWR072
+U 1 1 593FDB6D
+P 8150 1900
+F 0 "#PWR072" H 8150 1750 50  0001 C CNN
+F 1 "+BATT" H 8150 2040 50  0000 C CNN
+F 2 "" H 8150 1900 50  0001 C CNN
+F 3 "" H 8150 1900 50  0001 C CNN
+	1    8150 1900
+	1    0    0    -1
+$EndComp
+$Comp
+L +BATT #PWR073
+U 1 1 593FDC80
+P 8550 2150
+F 0 "#PWR073" H 8550 2000 50  0001 C CNN
+F 1 "+BATT" H 8550 2290 50  0000 C CNN
+F 2 "" H 8550 2150 50  0001 C CNN
+F 3 "" H 8550 2150 50  0001 C CNN
+	1    8550 2150
+	1    0    0    -1
+$EndComp
+Wire Wire Line
+	10550 3100 10300 3100
+Text Label 10550 3100 2    60   ~ 0
+IDX1
 $EndSCHEMATC

Commit message: control power to hall sensor from pld
Connections:
- net +BATT: no longer C23.1, R14.2, R15.1
- net ENL1: now also U10.10 (GPIO); no longer U10.11 (GPIO)
- net IDX: now also U10.11 (GPIO); no longer U10.12 (GPIO)
- net IDX1: now also U10.12 (GPIO); no longer U10.13 (GPIO)
- net LDO1: now also U10.9 (GPIO); no longer U10.10 (GPIO)
- new net TLV: C23.1, R14.2, R15.1, U10.13 (GPIO)
- no-connect marks 18 -> 17
Changed lines of the file:
@@
 Wire Wire Line
 	9150 3200 9400 3200
-Text Label 10550 3300 2    60   ~ 0
+Text Label 10550 3400 2    60   ~ 0
 ENL1
 Wire Wire Line
-	10550 3200 10300 3200
-Text Label 10550 3200 2    60   ~ 0
+	10550 3300 10300 3300
+Text Label 10550 3300 2    60   ~ 0
 IDX
 Wire Wire Line
-	10550 3300 10300 3300
+	10550 3400 10300 3400
 Text Label 10550 3000 2    60   ~ 0
 ENL
 Wire Wire Line
-	10550 3400 10300 3400
+	10550 3500 10300 3500
 Text Label 9150 3200 0    60   ~ 0
 LDO
@@
 Text Label 4650 1900 0    60   ~ 0
 LDO1
-Text Label 10550 3400 2    60   ~ 0
+Text Label 10550 3500 2    60   ~ 0
 LDO1
-NoConn ~ 10300 3500
 NoConn ~ 9400 3400
 NoConn ~ 9400 3500
@@
 NoConn ~ 4900 1800
 NoConn ~ 9400 3100
-$Comp
-L +BATT #PWR071
-U 1 1 593FCFD7
-P 7700 2150
-F 0 "#PWR071" H 7700 2000 50  0001 C CNN
-F 1 "+BATT" H 7700 2290 50  0000 C CNN
-F 2 "" H 7700 2150 50  0001 C CNN
-F 3 "" H 7700 2150 50  0001 C CNN
-	1    7700 2150
-	1    0    0    -1
-$EndComp
-$Comp
-L +BATT #PWR072
-U 1 1 593FDB6D
-P 8150 1900
-F 0 "#PWR072" H 8150 1750 50  0001 C CNN
-F 1 "+BATT" H 8150 2040 50  0000 C CNN
-F 2 "" H 8150 1900 50  0001 C CNN
-F 3 "" H 8150 1900 50  0001 C CNN
-	1    8150 1900
-	1    0    0    -1
-$EndComp
-$Comp
-L +BATT #PWR073
-U 1 1 593FDC80
-P 8550 2150
-F 0 "#PWR073" H 8550 2000 50  0001 C CNN
-F 1 "+BATT" H 8550 2290 50  0000 C CNN
-F 2 "" H 8550 2150 50  0001 C CNN
-F 3 "" H 8550 2150 50  0001 C CNN
-	1    8550 2150
-	1    0    0    -1
-$EndComp
 Wire Wire Line
-	10550 3100 10300 3100
+	10550 3200 10300 3200
+Text Label 10550 3200 2    60   ~ 0
+IDX1
+Wire Wire Line
+	10300 3100 10550 3100
 Text Label 10550 3100 2    60   ~ 0
-IDX1
+TLV
+Text Label 7850 2150 2    60   ~ 0
+TLV
+Text Label 8700 2150 2    60   ~ 0
+TLV
+Wire Wire Line
+	7850 2150 7700 2150
+Text Label 8300 1900 2    60   ~ 0
+TLV
+Wire Wire Line
+	8300 1900 8150 1900
+Wire Wire Line
+	8700 2150 8550 2150
 $EndSCHEMATC
